Commit message: TransportAviaryを追加

File: gym_pybullet_drones/assets/box_with_attachment.urdf (robot description, URDF)
Before this commit: robot box_with_attachments, 5 links, 4 joints
Links:
- link box_link: geometry collision box size=1.0 1.0 0.1; visual box size=1.0 1.0 0.1

File: gym_pybullet_drones/assets/connecting_rod.urdf (robot description, URDF)
Before this commit: robot connecting_rod, 3 links, 2 joints
Joints:
- joint drone_joint: axis (none) -> 0 0 1
